Commit message: my_robot_package

File: ros2_models/my_robot_description/urdf/my_robot.xacro (robot description, xacro)
@@ -2,4 +2,6 @@
 <robot name="my_robot"
   xmlns:xacro="http://www.ros.org/wiki/xacro">
+  <!-- add wheel xacro platform include files -->
+  <xacro:include filename="$(find my_robot_description)/urdf/wheel.xacro"/>
   <link name="base_link"></link>
   <joint name="base_link_joint" type="fixed">
@@ -10,11 +12,15 @@
   <link name='body_link'>
     <pose>0 0 0.1 0 0 0</pose>
+    <xacro:property name="mass" value="6" />
+    <xacro:property name="width" value="0.5" />
+    <xacro:property name="depth" value="0.7" />
+    <xacro:property name="height" value="0.2" />
     <inertial>
-      <mass value="5"/>
+      <mass value="${mass}"/>
       <origin xyz="0 0 0.05" rpy=" 0 0 0"/>
       <inertia
-      ixx="0.01" ixy="0.01" ixz="0"
-      iyy="0.01" iyz="0.01"
-      izz="0.01"
+      ixx="${1/12* mass*(width*width+height*height)}" ixy="0" ixz="0"
+      iyy="${1/12* mass*(depth*depth+height*height)}" iyz="0"
+      izz="${1/12* mass*(width*width+depth*depth)}"
       />
     </inertial>
@@ -22,5 +28,5 @@
       <origin xyz="0 0 0.02" rpy="0 0 0"/>
       <geometry>
-        <box size="0.4 0.2 0.1"/>
+        <mesh filename="package://my_robot_description/meshes/clearpath_husky_chassis.dae" scale="1 1 1"/>
       </geometry>
     </collision>
@@ -28,7 +34,16 @@
       <origin xyz="0 0 0.02" rpy=" 0 0 0"/>
       <geometry>
-        <box size="0.4 0.2 0.1"/>
+        <mesh filename="package://my_robot_description/meshes/clearpath_husky_chassis.dae" scale="1 1 1"/>
       </geometry>
     </visual>
   </link>
+   <!--wheel macros-->
+   <xacro:wheel alignment="front_left" x_="0.13" y_="-0.1" z_="0.0" r_="1.5707" p_="0" j_="0" >
+	</xacro:wheel>
+    <xacro:wheel alignment="front_right" x_="0.13" y_="0.1" z_="0.0" r_="1.5707" p_="0.0" j_="0.0" >
+	</xacro:wheel>
+   <xacro:wheel alignment="rear_left" x_="-0.13" y_="-0.1" z_="0.0" r_="1.5707" p_="0" j_="0" >
+	</xacro:wheel>
+    <xacro:wheel alignment="rear_right" x_="-0.13" y_="0.1" z_="0.0" r_="1.5707" p_="0.0" j_="0.0" >
+	</xacro:wheel>
 </robot>

Commit message: robot description package

File: ros2_models/my_robot_description/urdf/my_robot.xacro (robot description, xacro)
@@ -4,4 +4,6 @@
   <!-- add wheel xacro platform include files -->
   <xacro:include filename="$(find my_robot_description)/urdf/wheel.xacro"/>
+<!-- add gazebo plugins -->
+<xacro:include filename="$(find my_robot_description)/urdf/my_robot.gazebo"/>
   <link name="base_link"></link>
   <joint name="base_link_joint" type="fixed">
@@ -39,11 +41,45 @@
   </link>
    <!--wheel macros-->
-   <xacro:wheel alignment="front_left" x_="0.13" y_="-0.1" z_="0.0" r_="1.5707" p_="0" j_="0" >
+   <xacro:wheel alignment="front_left" x_="0.26" y_="-0.27" z_="0.03" r_="1.5707" p_="0" j_="0" >
 	</xacro:wheel>
-    <xacro:wheel alignment="front_right" x_="0.13" y_="0.1" z_="0.0" r_="1.5707" p_="0.0" j_="0.0" >
+    <xacro:wheel alignment="front_right" x_="0.26" y_="0.27" z_="0.03" r_="1.5707" p_="0.0" j_="0.0" >
 	</xacro:wheel>
-   <xacro:wheel alignment="rear_left" x_="-0.13" y_="-0.1" z_="0.0" r_="1.5707" p_="0" j_="0" >
+   <xacro:wheel alignment="rear_left" x_="-0.26" y_="-0.27" z_="0.03" r_="1.5707" p_="0" j_="0" >
 	</xacro:wheel>
-    <xacro:wheel alignment="rear_right" x_="-0.13" y_="0.1" z_="0.0" r_="1.5707" p_="0.0" j_="0.0" >
+    <xacro:wheel alignment="rear_right" x_="-0.26" y_="0.27" z_="0.03" r_="1.5707" p_="0.0" j_="0.0" >
 	</xacro:wheel>
+   <!-- rplidar Laser -->
+<link name="laser">
+  <collision>
+     <origin xyz="0 0 0" rpy="1.5707 0 4.71"/>
+     <geometry>
+       <mesh filename="package://my_robot_description/meshes/rplidar.stl" scale="0.001 0.001 0.001" />
+     </geometry>
+   </collision>
+   <visual>
+     <origin xyz="0 0 0" rpy="1.5707 0 4.71"/>
+     <geometry>
+     <mesh filename="package://my_robot_description/meshes/rplidar.stl" scale="0.001 0.001 0.001" />
+     </geometry>
+   </visual>
+   <inertial>
+     <mass value="1e-5" />
+     <origin xyz="0 0 0" rpy="1.5707 0 4.71"/>
+       <inertia ixx="0" ixy="0" ixz="0" iyy="0" iyz="0" izz="0" />
+      </inertial>
+ </link>
+ <joint name="rplidar_joint" type="fixed">
+    <axis xyz="0 1 0" />
+     <origin xyz="0.23 0 0.24" rpy="0 0 3.14"/>
+    <parent link="body_link"/>
+    <child link="laser"/>
+ </joint>
+<!--imu-->
+ <joint name="imu_joint" type="fixed">
+    <origin xyz="0 0 0" rpy="0 0 0"/>
+    <parent link="body_link"/>
+    <child link="imu_link"/>
+  </joint>
+  <link name="imu_link">
+  </link>
 </robot>

File: ros2_models/my_robot_description/urdf/wheel.xacro (robot description, xacro)
@@ -4,6 +4,6 @@
                 <link name="${alignment}_wheel">
                             <xacro:property name="w_mass" value="0.5" />
-                            <xacro:property name="w_radius" value="0.1" />
-                            <xacro:property name="w_height" value="0.05" />
+                            <xacro:property name="w_radius" value="0.15" />
+                            <xacro:property name="w_height" value="0.1" />
                         <visual>
                                 <origin xyz="0 0 0" rpy="${r_} 0 0"/>
