Commit message: modified:   ros2_models/my_robot_description/urdf/my_robot.gazebo 	modified:   ros2_models/my_robot_description/urdf/wheel.xacro

File: ros2_models/my_robot_description/urdf/wheel.xacro (robot description, xacro)
@@ -43,4 +43,13 @@
                    <material>Gazebo/Black</material>
                 </gazebo>
+                <transmission name="${alignment}_wheel_trans" type="SimpleTransmission">
+                <type>transmission_interface/SimpleTransmission</type>
+                   <actuator name="${alignment}_wheel_motor">
+                     <mechanicalReduction>1</mechanicalReduction>
+                   </actuator>
+                 <joint name="${alignment}_wheel_hinge">
+             <hardwareInterface>hardware_interface/EffortJointInterface</hardwareInterface>
+                   </joint>
+                </transmission>
         </xacro:macro>
 </robot>
